Commit message: single arm hand tracking is working

File: assets/universal_robots_ur5e/dual_ur5e.urdf (robot description, URDF)
Before this commit: robot dual_ur5e_robot, 23 links, 22 joints
Joints:
- joint world_to_left_arm_base: origin xyz=0 0.275 0.3 rpy=0.7853981633974483 0 3.141592653589793 -> xyz=0 0.275 0 rpy=0 0 0
- joint world_to_right_arm_base: origin xyz=0 -0.275 0.3 rpy=0.7853981633974483 0 0 -> xyz=0 -0.275 0 rpy=0 0 0

Commit message: robot arm rotation success

File: assets/universal_robots_ur5e/dual_ur5e.urdf (robot description, URDF)
Before this commit: robot dual_ur5e_robot, 23 links, 22 joints
Joints:
- joint world_to_left_arm_base: origin xyz=0 0.275 0.3 rpy=0.7853981633974483 0 3.141592653589793 -> xyz=0 0.275 0.3 rpy=0 0 0

Commit message: Correct Rotation now

File: assets/universal_robots_ur5e/dual_ur5e.urdf (robot description, URDF)
Before this commit: robot dual_ur5e_robot, 23 links, 22 joints
Joints:
- joint world_to_left_arm_base: origin xyz=0 0.275 0.3 rpy=0 0 0 -> xyz=0 0.275 0.3 rpy=0 0 3.141592653589793

Commit message: Correct Transform for both arms

File: assets/universal_robots_ur5e/dual_ur5e.urdf (robot description, URDF)
Before this commit: robot dual_ur5e_robot, 23 links, 22 joints
Joints:
- joint world_to_left_arm_base: origin xyz=0 0.275 0.3 rpy=0 0 3.141592653589793 -> xyz=0 0.275 0 rpy=0 0 3.141592653589793
- joint world_to_right_arm_base: origin xyz=0 -0.275 0.3 rpy=0.7853981633974483 0 0 -> xyz=0 -0.275 0 rpy=0 0 0

Commit message: Better

File: assets/universal_robots_ur5e/dual_ur5e.urdf (robot description, URDF)
Before this commit: robot dual_ur5e_robot, 23 links, 22 joints
Joints:
- joint world_to_left_arm_base: origin xyz=0 0.275 0 rpy=0 0 0 -> xyz=0 0.275 0 rpy=0 0 3.141592653589793
